Commit message: update hierarki

File: rscuad_description/urdf/rscuad.xacro (robot description, xacro)
@@ -4,10 +4,7 @@
      For more information, please see http://wiki.ros.org/sw_urdf_exporter -->
 <robot name="rscuad" xmlns:xacro="http://www.ros.org/wiki/xacro">
+  <xacro:property name="PI" value="3.1415926535897931"/>
   <xacro:include filename="$(find rscuad)/urdf/rscuad.gazebo" />
-  <gazebo>
-    <plugin name="gazebo_ros_control" filename="libgazebo_ros_control.so">
-      <robotNamespace>/rscuad</robotNamespace>
-    </plugin>
-  </gazebo>
+  <xacro:include filename="$(find rscuad)/urdf/transmission.xacro" />
   <link
     name="body">
@@ -108,14 +105,5 @@
       velocity="0" />
   </joint>
-  <transmission name="head_pan_trans">
-    <type>transmission_interface/SimpleTransmission</type>
-    <joint name="head_pan">
-      <hardwareInterface>EffortJointInterface</hardwareInterface>
-    </joint>
-    <actuator name="head_pan_motor">
-      <hardwareInterface>EffortJointInterface</hardwareInterface>
-      <mechanicalReduction>1</mechanicalReduction>
-    </actuator>
-  </transmission>
+  <transmissions joint="head_pan"/>
   <link
     name="head_tilt">
@@ -176,14 +164,5 @@
       velocity="0" />
   </joint>
-  <transmission name="head_tilt_trans">
-    <type>transmission_interface/SimpleTransmission</type>
-    <joint name="head_tilt">
-      <hardwareInterface>EffortJointInterface</hardwareInterface>
-    </joint>
-    <actuator name="head_tilt_motor">
-      <hardwareInterface>EffortJointInterface</hardwareInterface>
-      <mechanicalReduction>1</mechanicalReduction>
-    </actuator>
-  </transmission>
+  <transmissions joint="head_tilt"/>
   <link
     name="l_sho_pitch">
@@ -244,4 +223,5 @@
       velocity="0" />
   </joint>
+  <transmissions joint="l_sho_pitch"/>
   <link
     name="l_sho_roll">
@@ -302,4 +282,5 @@
       velocity="0" />
   </joint>
+  <transmissions joint="l_sho_roll"/>
   <link
     name="l_el">
@@ -360,4 +341,5 @@
       velocity="0" />
   </joint>
+  <transmissions joint="l_el"/>
   <link
     name="r_sho_pitch">
@@ -418,4 +400,5 @@
       velocity="0" />
   </joint>
+  <transmissions joint="r_sho_pitch"/>
   <link
     name="r_sho_roll">
@@ -476,4 +459,5 @@
       velocity="0" />
   </joint>
+  <transmissions joint="r_sho_roll"/>
   <link
     name="r_el">
@@ -534,4 +518,5 @@
       velocity="0" />
   </joint>
+  <transmissions joint="r_el"/>
   <link
     name="l_hip_yaw">
@@ -592,4 +577,5 @@
       velocity="0" />
   </joint>
+  <transmissions joint="l_hip_yaw"/>
   <link
     name="l_hip_roll">
@@ -650,4 +636,5 @@
       velocity="0" />
   </joint>
+  <transmissions joint="l_hip_roll"/>
   <link
     name="l_hip_pitch">
@@ -708,4 +695,5 @@
       velocity="0" />
   </joint>
+  <transmissions joint="l_hip_pitch"/>
   <link
     name="l_knee">
@@ -766,4 +754,5 @@
       velocity="0" />
   </joint>
+  <transmissions joint="l_knee"/>
   <link
     name="l_ank_pitch">
@@ -824,4 +813,5 @@
       velocity="0" />
   </joint>
+  <transmissions joint="l_ank_pitch"/>
   <link
     name="l_ank_roll">
@@ -882,4 +872,5 @@
       velocity="0" />
   </joint>
+  <transmissions joint="l_ank_roll"/>
   <link
     name="r_hip_yaw">
@@ -940,4 +931,5 @@
       velocity="0" />
   </joint>
+  <transmissions joint="r_hip_yaw"/>
   <link
     name="r_hip_roll">
@@ -998,4 +990,5 @@
       velocity="0" />
   </joint>
+  <transmissions joint="r_hip_roll"/>
   <link
     name="r_hip_pitch">
@@ -1056,4 +1049,5 @@
       velocity="0" />
   </joint>
+  <transmissions joint="r_hip_pitch"/>
   <link
     name="r_knee">
@@ -1114,4 +1108,5 @@
       velocity="0" />
   </joint>
+  <transmissions joint="r_knee"/>
   <link
     name="r_ank_pitch">
@@ -1172,4 +1167,5 @@
       velocity="0" />
   </joint>
+  <transmissions joint="r_ank_pitch"/>
   <link
     name="r_ank_roll">
@@ -1230,3 +1226,4 @@
       velocity="0" />
   </joint>
+  <transmissions joint="r_ank_roll"/>
 </robot>

Commit message: update structure

File: rscuad_description/urdf/rscuad.xacro (robot description, xacro)
@@ -105,5 +105,5 @@
       velocity="0" />
   </joint>
-  <transmissions joint="head_pan"/>
+  <insert_transmission name="head_pan"/>
   <link
     name="head_tilt">
@@ -164,5 +164,5 @@
       velocity="0" />
   </joint>
-  <transmissions joint="head_tilt"/>
+  <insert_transmission name="head_tilt"/>
   <link
     name="l_sho_pitch">
@@ -220,8 +220,8 @@
       lower="0"
       upper="0"
-      effort="0"
-      velocity="0" />
-  </joint>
-  <transmissions joint="l_sho_pitch"/>
+      effort="100"
+      velocity="1000" />
+  </joint>
+  <insert_transmission name="l_sho_pitch"/>
   <link
     name="l_sho_roll">
@@ -282,5 +282,5 @@
       velocity="0" />
   </joint>
-  <transmissions joint="l_sho_roll"/>
+  <insert_transmission name="l_sho_roll"/>
   <link
     name="l_el">
@@ -341,5 +341,5 @@
       velocity="0" />
   </joint>
-  <transmissions joint="l_el"/>
+  <insert_transmission name="l_el"/>
   <link
     name="r_sho_pitch">
@@ -400,5 +400,5 @@
       velocity="0" />
   </joint>
-  <transmissions joint="r_sho_pitch"/>
+  <insert_transmission name="r_sho_pitch"/>
   <link
     name="r_sho_roll">
@@ -459,5 +459,5 @@
       velocity="0" />
   </joint>
-  <transmissions joint="r_sho_roll"/>
+  <insert_transmission name="r_sho_roll"/>
   <link
     name="r_el">
@@ -518,5 +518,5 @@
       velocity="0" />
   </joint>
-  <transmissions joint="r_el"/>
+  <insert_transmission name="r_el"/>
   <link
     name="l_hip_yaw">
@@ -577,5 +577,5 @@
       velocity="0" />
   </joint>
-  <transmissions joint="l_hip_yaw"/>
+  <insert_transmission name="l_hip_yaw"/>
   <link
     name="l_hip_roll">
@@ -636,5 +636,5 @@
       velocity="0" />
   </joint>
-  <transmissions joint="l_hip_roll"/>
+  <insert_transmission name="l_hip_roll"/>
   <link
     name="l_hip_pitch">
@@ -695,5 +695,5 @@
       velocity="0" />
   </joint>
-  <transmissions joint="l_hip_pitch"/>
+  <insert_transmission name="l_hip_pitch"/>
   <link
     name="l_knee">
@@ -754,5 +754,5 @@
       velocity="0" />
   </joint>
-  <transmissions joint="l_knee"/>
+  <insert_transmission name="l_knee"/>
   <link
     name="l_ank_pitch">
@@ -813,5 +813,5 @@
       velocity="0" />
   </joint>
-  <transmissions joint="l_ank_pitch"/>
+  <insert_transmission name="l_ank_pitch"/>
   <link
     name="l_ank_roll">
@@ -872,5 +872,5 @@
       velocity="0" />
   </joint>
-  <transmissions joint="l_ank_roll"/>
+  <insert_transmission name="l_ank_roll"/>
   <link
     name="r_hip_yaw">
@@ -931,5 +931,5 @@
       velocity="0" />
   </joint>
-  <transmissions joint="r_hip_yaw"/>
+  <insert_transmission name="r_hip_yaw"/>
   <link
     name="r_hip_roll">
@@ -990,5 +990,5 @@
       velocity="0" />
   </joint>
-  <transmissions joint="r_hip_roll"/>
+  <insert_transmission name="r_hip_roll"/>
   <link
     name="r_hip_pitch">
@@ -1049,5 +1049,5 @@
       velocity="0" />
   </joint>
-  <transmissions joint="r_hip_pitch"/>
+  <insert_transmission name="r_hip_pitch"/>
   <link
     name="r_knee">
@@ -1108,5 +1108,5 @@
       velocity="0" />
   </joint>
-  <transmissions joint="r_knee"/>
+  <insert_transmission name="r_knee"/>
   <link
     name="r_ank_pitch">
@@ -1167,5 +1167,5 @@
       velocity="0" />
   </joint>
-  <transmissions joint="r_ank_pitch"/>
+  <insert_transmission name="r_ank_pitch"/>
   <link
     name="r_ank_roll">
@@ -1226,4 +1226,4 @@
       velocity="0" />
   </joint>
-  <transmissions joint="r_ank_roll"/>
+  <insert_transmission name="r_ank_roll"/>
 </robot>

File: rscuad_description/urdf/transmission.xacro (robot description, xacro)
@@ -1,15 +1,15 @@
 <?xml version="1.0" ?>
-    <robot name="rscuad">
-        <macro name="transmissions" params="joint">
-            <transmission name="${joint}_trans">
-                <type>transmission_interface/SimpleTransmission</type>
-                <joint name="${joint}">
-                <hardwareInterface>EffortJointInterface</hardwareInterface>
-                </joint>
-                <actuator name="${joint}_motor">
-                <hardwareInterface>EffortJointInterface</hardwareInterface>
-                <mechanicalReduction>1</mechanicalReduction>
-                </actuator>
-            </transmission>
-        </macro>
-    </robot>
+  <robot xmlns:xacro="http://ros.org/wiki/xacro">
+  <xacro:macro name="insert_transmission" params="name">
+    <transmission name="${name}_tran">
+      <type>transmission_interface/SimpleTransmission</type>
+      <joint name="${name}">
+        <hardwareInterface>hardware_interface/EffortJointInterface</hardwareInterface>
+      </joint>
+      <actuator name="${name}_motor">
+        <hardwareInterface>hardware_interface/EffortJointInterface</hardwareInterface>
+        <mechanicalReduction>1</mechanicalReduction>
+      </actuator>
+    </transmission>
+  </xacro:macro>
+</robot>

Commit message: update all join

File: rscuad_description/urdf/rscuad.xacro (robot description, xacro)
@@ -5,6 +5,6 @@
 <robot name="rscuad" xmlns:xacro="http://www.ros.org/wiki/xacro">
   <xacro:property name="PI" value="3.1415926535897931"/>
-  <xacro:include filename="$(find rscuad)/urdf/rscuad.gazebo" />
-  <xacro:include filename="$(find rscuad)/urdf/transmission.xacro" />
+  <xacro:include filename="$(find rscuad_description)/urdf/rscuad.gazebo" />
+  <xacro:include filename="$(find rscuad_description)/urdf/transmission.xacro" />
   <link
     name="body">
@@ -29,19 +29,19 @@
       <geometry>
         <mesh
-          filename="package://rscuad/meshes/body.STL" />
-      </geometry>
-      <material
-        name="">
-        <color
-          rgba="0.752941176470588 0.752941176470588 0.752941176470588 1" />
-      </material>
-    </visual>
-    <collision>
-      <origin
-        xyz="0 0 0"
-        rpy="0 0 0" />
-      <geometry>
-        <mesh
-          filename="package://rscuad/meshes/body.STL" />
+          filename="package://rscuad_description/meshes/body.STL" />
+      </geometry>
+      <material
+        name="">
+        <color
+          rgba="0.752941176470588 0.752941176470588 0.752941176470588 1" />
+      </material>
+    </visual>
+    <collision>
+      <origin
+        xyz="0 0 0"
+        rpy="0 0 0" />
+      <geometry>
+        <mesh
+          filename="package://rscuad_description/meshes/body.STL" />
       </geometry>
     </collision>
@@ -69,5 +69,5 @@
       <geometry>
         <mesh
-          filename="package://rscuad/meshes/head_pan.STL" />
+          filename="package://rscuad_description/meshes/head_pan.STL" />
       </geometry>
       <material
@@ -83,5 +83,5 @@
       <geometry>
         <mesh
-          filename="package://rscuad/meshes/head_pan.STL" />
+          filename="package://rscuad_description/meshes/head_pan.STL" />
       </geometry>
     </collision>
@@ -128,19 +128,19 @@
       <geometry>
         <mesh
-          filename="package://rscuad/meshes/head_tilt.STL" />
-      </geometry>
-      <material
-        name="">
-        <color
-          rgba="0.752941176470588 0.752941176470588 0.752941176470588 1" />
-      </material>
-    </visual>
-    <collision>
-      <origin
-        xyz="0 0 0"
-        rpy="0 0 0" />
-      <geometry>
-        <mesh
-          filename="package://rscuad/meshes/head_tilt.STL" />
+          filename="package://rscuad_description/meshes/head_tilt.STL" />
+      </geometry>
+      <material
+        name="">
+        <color
+          rgba="0.752941176470588 0.752941176470588 0.752941176470588 1" />
+      </material>
+    </visual>
+    <collision>
+      <origin
+        xyz="0 0 0"
+        rpy="0 0 0" />
+      <geometry>
+        <mesh
+          filename="package://rscuad_description/meshes/head_tilt.STL" />
       </geometry>
     </collision>
@@ -165,4 +165,5 @@
   </joint>
   <insert_transmission name="head_tilt"/>
+<!-- ================================================ hand left -->
   <link
     name="l_sho_pitch">
@@ -187,19 +188,19 @@
       <geometry>
         <mesh
-          filename="package://rscuad/meshes/l_sho_pitch.STL" />
-      </geometry>
-      <material
-        name="">
-        <color
-          rgba="0.752941176470588 0.752941176470588 0.752941176470588 1" />
-      </material>
-    </visual>
-    <collision>
-      <origin
-        xyz="0 0 0"
-        rpy="0 0 0" />
-      <geometry>
-        <mesh
-          filename="package://rscuad/meshes/l_sho_pitch.STL" />
+          filename="package://rscuad_description/meshes/l_sho_pitch.STL" />
+      </geometry>
+      <material
+        name="">
+        <color
+          rgba="0.752941176470588 0.752941176470588 0.752941176470588 1" />
+      </material>
+    </visual>
+    <collision>
+      <origin
+        xyz="0 0 0"
+        rpy="0 0 0" />
+      <geometry>
+        <mesh
+          filename="package://rscuad_description/meshes/l_sho_pitch.STL" />
       </geometry>
     </collision>
@@ -207,5 +208,5 @@
   <joint
     name="l_sho_pitch"
-    type="revolute">
+    type="continuous">
     <origin
       xyz="0.10096 -0.1394 0.12423"
@@ -246,19 +247,19 @@
       <geometry>
         <mesh
-          filename="package://rscuad/meshes/l_sho_roll.STL" />
-      </geometry>
-      <material
-        name="">
-        <color
-          rgba="0.752941176470588 0.752941176470588 0.752941176470588 1" />
-      </material>
-    </visual>
-    <collision>
-      <origin
-        xyz="0 0 0"
-        rpy="0 0 0" />
-      <geometry>
-        <mesh
-          filename="package://rscuad/meshes/l_sho_roll.STL" />
+          filename="package://rscuad_description/meshes/l_sho_roll.STL" />
+      </geometry>
+      <material
+        name="">
+        <color
+          rgba="0.752941176470588 0.752941176470588 0.752941176470588 1" />
+      </material>
+    </visual>
+    <collision>
+      <origin
+        xyz="0 0 0"
+        rpy="0 0 0" />
+      <geometry>
+        <mesh
+          filename="package://rscuad_description/meshes/l_sho_roll.STL" />
       </geometry>
     </collision>
@@ -266,5 +267,5 @@
   <joint
     name="l_sho_roll"
-    type="revolute">
+    type="continuous">
     <origin
       xyz="0.0385 -0.01 0"
@@ -279,5 +280,5 @@
       lower="0"
       upper="0"
-      effort="0"
+      effort="1000"
       velocity="0" />
   </joint>
@@ -305,19 +306,19 @@
       <geometry>
         <mesh
-          filename="package://rscuad/meshes/l_el.STL" />
-      </geometry>
-      <material
-        name="">
-        <color
-          rgba="0.752941176470588 0.752941176470588 0.752941176470588 1" />
-      </material>
-    </visual>
-    <collision>
-      <origin
-        xyz="0 0 0"
-        rpy="0 0 0" />
-      <geometry>
-        <mesh
-          filename="package://rscuad/meshes/l_el.STL" />
+          filename="package://rscuad_description/meshes/l_el.STL" />
+      </geometry>
+      <material
+        name="">
+        <color
+          rgba="0.752941176470588 0.752941176470588 0.752941176470588 1" />
+      </material>
+    </visual>
+    <collision>
+      <origin
+        xyz="0 0 0"
+        rpy="0 0 0" />
+      <geometry>
+        <mesh
+          filename="package://rscuad_description/meshes/l_el.STL" />
       </geometry>
     </collision>
@@ -325,5 +326,5 @@
   <joint
     name="l_el"
-    type="revolute">
+    type="continuous">
     <origin
       xyz="0.0874466726391421 0 0.0100000000000002"
@@ -338,8 +339,9 @@
       lower="0"
       upper="0"
-      effort="0"
+      effort="1000"
       velocity="0" />
   </joint>
   <insert_transmission name="l_el"/>
+<!-- ================================================ hand right -->
   <link
     name="r_sho_pitch">
@@ -364,19 +366,19 @@
       <geometry>
         <mesh
-          filename="package://rscuad/meshes/r_sho_pitch.STL" />
-      </geometry>
-      <material
-        name="">
-        <color
-          rgba="0.752941176470588 0.752941176470588 0.752941176470588 1" />
-      </material>
-    </visual>
-    <collision>
-      <origin
-        xyz="0 0 0"
-        rpy="0 0 0" />
-      <geometry>
-        <mesh
-          filename="package://rscuad/meshes/r_sho_pitch.STL" />
+          filename="package://rscuad_description/meshes/r_sho_pitch.STL" />
+      </geometry>
+      <material
+        name="">
+        <color
+          rgba="0.752941176470588 0.752941176470588 0.752941176470588 1" />
+      </material>
+    </visual>
+    <collision>
+      <origin
+        xyz="0 0 0"
+        rpy="0 0 0" />
+      <geometry>
+        <mesh
+          filename="package://rscuad_description/meshes/r_sho_pitch.STL" />
       </geometry>
     </collision>
@@ -384,5 +386,5 @@
   <joint
     name="r_sho_pitch"
-    type="revolute">
+    type="continuous">
     <origin
       xyz="-0.0290205030447131 -0.139400454049433 0.124229542783902"
@@ -397,5 +399,5 @@
       lower="0"
       upper="0"
-      effort="0"
+      effort="1000"
       velocity="0" />
   </joint>
@@ -423,19 +425,19 @@
       <geometry>
         <mesh
-          filename="package://rscuad/meshes/r_sho_roll.STL" />
-      </geometry>
-      <material
-        name="">
-        <color
-          rgba="0.752941176470588 0.752941176470588 0.752941176470588 1" />
-      </material>
-    </visual>
-    <collision>
-      <origin
-        xyz="0 0 0"
-        rpy="0 0 0" />
-      <geometry>
-        <mesh
-          filename="package://rscuad/meshes/r_sho_roll.STL" />
+          filename="package://rscuad_description/meshes/r_sho_roll.STL" />
+      </geometry>
+      <material
+        name="">
+        <color
+          rgba="0.752941176470588 0.752941176470588 0.752941176470588 1" />
+      </material>
+    </visual>
+    <collision>
+      <origin
+        xyz="0 0 0"
+        rpy="0 0 0" />
+      <geometry>
+        <mesh
+          filename="package://rscuad_description/meshes/r_sho_roll.STL" />
       </geometry>
     </collision>
@@ -443,5 +445,5 @@
   <joint
     name="r_sho_roll"
-    type="revolute">
+    type="continuous">
     <origin
       xyz="-0.0384999999999999 -0.00999999999999629 0"
@@ -456,5 +458,5 @@
       lower="0"
       upper="0"
-      effort="0"
+      effort="1000"
       velocity="0" />
   </joint>
@@ -482,19 +484,19 @@
       <geometry>
         <mesh
-          filename="package://rscuad/meshes/r_el.STL" />
-      </geometry>
-      <material
-        name="">
-        <color
-          rgba="0.752941176470588 0.752941176470588 0.752941176470588 1" />
-      </material>
-    </visual>
-    <collision>
-      <origin
-        xyz="0 0 0"
-        rpy="0 0 0" />
-      <geometry>
-        <mesh
-          filename="package://rscuad/meshes/r_el.STL" />
+          filename="package://rscuad_description/meshes/r_el.STL" />
+      </geometry>
+      <material
+        name="">
+        <color
+          rgba="0.752941176470588 0.752941176470588 0.752941176470588 1" />
+      </material>
+    </visual>
+    <collision>
+      <origin
+        xyz="0 0 0"
+        rpy="0 0 0" />
+      <geometry>
+        <mesh
+          filename="package://rscuad_description/meshes/r_el.STL" />
       </geometry>
     </collision>
@@ -502,5 +504,5 @@
   <joint
     name="r_el"
-    type="revolute">
+    type="continuous">
     <origin
       xyz="-0.0936500000000009 0 0.0099999999999961"
@@ -515,8 +517,9 @@
       lower="0"
       upper="0"
-      effort="0"
+      effort="1000"
       velocity="0" />
   </joint>
   <insert_transmission name="r_el"/>
+<!-- =====================================================leg left -->
   <link
     name="l_hip_yaw">
@@ -541,19 +544,19 @@
       <geometry>
         <mesh
-          filename="package://rscuad/meshes/l_hip_yaw.STL" />
-      </geometry>
-      <material
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