Commit message: leg approach not fix

File: rscuad_description/urdf/rscuad.xacro (robot description, xacro)
@@ -15,11 +15,7 @@
       <mass
         value="0.845681147773924" />
-      <inertia
-        ixx="0.000942220952716164"
-        ixy="-2.09951911714263E-09"
-        ixz="-5.82097094435726E-08"
-        iyy="0.0017318252778068"
-        iyz="-1.03521875266935E-06"
-        izz="0.00124711287069091" />
+      <inertia ixx="0.00340499" ixy="0.00000572" ixz="-0.00004256"
+             iyy="0.00296939" iyz="-0.00000059"
+             izz="0.00317331" />
     </inertial>
     <visual>
@@ -55,11 +51,7 @@
       <mass
         value="0.0127468700670499" />
-      <inertia
-        ixx="1.79344391432726E-06"
-        ixy="-2.0975806235736E-19"
-        ixz="-6.00252605549835E-20"
-        iyy="4.1896342976115E-06"
-        iyz="3.39828602459364E-07"
-        izz="4.30251924868049E-06" />
+      <inertia ixx="0.00000397" ixy="0.0" ixz="-0.00000031"
+             iyy="0.00000165" iyz="0.0"
+             izz="0.00000387" />
     </inertial>
     <visual>
@@ -103,5 +95,5 @@
       upper="0"
       effort="50"
-      velocity="0" />
+      velocity="0.1" />
   </joint>
   <insert_transmission name="head_pan"/>
@@ -114,11 +106,7 @@
       <mass
         value="0.12573924511903" />
-      <inertia
-        ixx="4.42942214862057E-05"
-        ixy="1.33185070586968E-08"
-        ixz="-1.54689849752873E-08"
-        iyy="5.02585908476386E-05"
-        iyz="-4.89972787819791E-08"
-        izz="4.4092437431138E-05" />
+      <inertia ixx="0.00010612" ixy="0.00000011" ixz="-0.00000910"
+             iyy="0.00008721" iyz="0.00000084"
+             izz="0.00004529" />
     </inertial>
     <visual>
@@ -162,5 +150,5 @@
       upper="0"
       effort="50"
-      velocity="0" />
+      velocity="0.1" />
   </joint>
   <insert_transmission name="head_tilt"/>
@@ -174,11 +162,7 @@
       <mass
         value="0.016476449424892" />
-      <inertia
-        ixx="4.47813381956679E-06"
-        ixy="3.39828602459356E-07"
-        ixz="1.79079949513068E-19"
-        iyy="4.47784883764015E-06"
-        iyz="6.04884335805419E-20"
-        izz="1.96877350328692E-06" />
+      <inertia ixx="0.00000165" ixy="0.0" ixz="0.0"
+             iyy="0.00000387" iyz="0.00000031"
+             izz="0.00000397" />
     </inertial>
     <visual>
@@ -222,5 +206,5 @@
       upper="0"
       effort="100"
-      velocity="1000" />
+      velocity="0.1" />
   </joint>
   <insert_transmission name="l_sho_pitch"/>
@@ -233,11 +217,7 @@
       <mass
         value="0.0884003305596694" />
-      <inertia
-        ixx="1.54544096501495E-05"
-        ixy="2.90930703710243E-07"
-        ixz="-3.1936718627683E-07"
-        iyy="1.80602730144738E-05"
-        iyz="3.0377515300486E-13"
-        izz="1.77147455885611E-05" />
+      <inertia ixx="0.00022804" ixy="-0.00000001" ixz="0.00000003"
+             iyy="0.00003042" iyz="0.00000059"
+             izz="0.00023474" />
     </inertial>
     <visual>
@@ -281,5 +261,5 @@
       upper="0"
       effort="1000"
-      velocity="0" />
+      velocity="0.1" />
   </joint>
   <insert_transmission name="l_sho_roll"/>
@@ -292,11 +272,7 @@
       <mass
         value="0.0561826372694756" />
-      <inertia
-        ixx="2.9049589881886E-05"
-        ixy="2.03830392463693E-08"
-        ixz="3.79159526035902E-07"
-        iyy="3.38921458240999E-05"
-        iyz="1.12947145945233E-14"
-        izz="1.34693310072719E-05" />
+      <inertia ixx="0.00006196" ixy="0.0" ixz="0.0"
+             iyy="0.00001231" iyz="-0.00000372"
+             izz="0.00006854" />
     </inertial>
     <visual>
@@ -340,5 +316,5 @@
       upper="0"
       effort="1000"
-      velocity="0" />
+      velocity="0.1" />
   </joint>
   <insert_transmission name="l_el"/>
@@ -352,11 +328,7 @@
       <mass
         value="0.0164764494248921" />
-      <inertia
-        ixx="4.4781338195668E-06"
-        ixy="-3.39828602459362E-07"
-        ixz="2.01210430228637E-19"
-        iyy="4.47784883764016E-06"
-        iyz="-5.87818990239026E-20"
-        izz="1.96877350328693E-06" />
+      <inertia ixx="0.00000165" ixy="0.0" ixz="0.0"
+             iyy="0.00000387" iyz="-0.00000031"
+             izz="0.00000397" />
     </inertial>
     <visual>
@@ -400,5 +372,5 @@
       upper="0"
       effort="1000"
-      velocity="0" />
+      velocity="0.1" />
   </joint>
   <insert_transmission name="r_sho_pitch"/>
@@ -411,11 +383,7 @@
       <mass
         value="0.0884003307974895" />
-      <inertia
-        ixx="1.54544096503321E-05"
-        ixy="-2.90930609797706E-07"
-        ixz="3.19523950275379E-07"
-        iyy="1.8060273013059E-05"
-        iyz="-3.03961651424894E-13"
-        izz="1.7714745586952E-05" />
+      <inertia ixx="0.00022804" ixy="0.00000001" ixz="0.00000003"
+             iyy="0.00003042" iyz="-0.00000059"
+             izz="0.00023474" />
     </inertial>
     <visual>
@@ -459,5 +427,5 @@
       upper="0"
       effort="1000"
-      velocity="0" />
+      velocity="0.1" />
   </joint>
   <insert_transmission name="r_sho_roll"/>
@@ -470,11 +438,7 @@
       <mass
         value="0.0561826372694755" />
-      <inertia
-        ixx="2.90495898818859E-05"
-        ixy="-2.03830290064609E-08"
-        ixz="-3.79159620555639E-07"
-        iyy="3.38921458240998E-05"
-        iyz="-1.12946351407492E-14"
-        izz="1.34693310072719E-05" />
+      <inertia ixx="0.00006196" ixy="0.0" ixz="0.0"
+             iyy="0.00001231" iyz="0.00000372"
+             izz="0.00006854" />
     </inertial>
     <visual>
@@ -518,5 +482,5 @@
       upper="0"
       effort="1000"
-      velocity="0" />
+      velocity="0.1" />
   </joint>
   <insert_transmission name="r_el"/>
@@ -530,11 +494,7 @@
       <mass
         value="0.0229829364852389" />
-      <inertia
-        ixx="1.43427059428117E-05"
-        ixy="8.27728850430916E-11"
-        ixz="1.78618118574046E-10"
-        iyy="1.40196878929158E-05"
-        iyz="3.77243123517952E-08"
-        izz="5.34102862853241E-06" />
+      <inertia ixx="0.00000151" ixy="0.0" ixz="0.00000001"
+             iyy="0.00000430" iyz="0.0"
+             izz="0.00000412" />
     </inertial>
     <visual>
@@ -578,5 +538,5 @@
       upper="0"
       effort="1000"
-      velocity="0" />
+      velocity="0.1" />
   </joint>
   <insert_transmission name="l_hip_yaw"/>
@@ -589,11 +549,7 @@
       <mass
         value="0.151586182496668" />
-      <inertia
-        ixx="5.5028175022932E-05"
-        ixy="-8.98410976515644E-07"
-        ixz="1.16956229470377E-12"
-        iyy="3.44253544650063E-05"
-        iyz="-9.07683611385409E-07"
-        izz="5.54170402685468E-05" />
+      <inertia ixx="0.00004661" ixy="-0.00000101" ixz="-0.00000131"
+             iyy="0.00012523" iyz="-0.00000006"
+             izz="0.00010857" />
     </inertial>
     <visual>
@@ -637,5 +593,5 @@
       upper="0"
       effort="1000"
-      velocity="0" />
+      velocity="0.1" />
   </joint>
   <insert_transmission name="l_hip_roll"/>
@@ -648,11 +604,7 @@
       <mass
         value="0.100631639038866" />
-      <inertia
-        ixx="4.17310749465033E-05"
-        ixy="8.88098878734448E-07"
-        ixz="5.42245635048738E-09"
-        iyy="3.2141171755086E-05"
-        iyz="6.05524366448529E-07"
-        izz="5.70627485423253E-05" />
+      <inertia ixx="0.00010499" ixy="-0.00000001" ixz="-0.00000071"
+             iyy="0.00009613" iyz="0.00000353"
+             izz="0.00002493" />
     </inertial>
     <visual>
@@ -696,5 +648,5 @@
       upper="0"
       effort="1000"
-      velocity="0" />
+      velocity="0.1" />
   </joint>
   <insert_transmission name="l_hip_pitch"/>
@@ -707,11 +659,7 @@
       <mass
         value="0.0624359207391482" />
-      <inertia
-        ixx="0.000103909612579584"
-        ixy="2.24696234615877E-10"
-        ixz="1.61509844645296E-10"
-        iyy="4.75106496264908E-05"
-        iyz="-1.78798066876229E-05"
-        izz="0.000119654238933631" />
+      <inertia ixx="0.00003715" ixy="0.0" ixz="0.0"
+             iyy="0.00002751" iyz="0.0"
+             izz="0.00001511" />
     </inertial>
     <visual>
@@ -755,5 +703,5 @@
       upper="0"
       effort="1000"
-      velocity="0" />
+      velocity="0.1" />
   </joint>
   <insert_transmission name="l_knee"/>
@@ -766,11 +714,7 @@
       <mass
         value="0.151586182496668" />
-      <inertia
-        ixx="5.50281750229324E-05"
-        ixy="8.98440761834264E-07"
-        ixz="1.16956223612234E-12"
-        iyy="3.44253544650064E-05"
-        iyz="-9.07656515072525E-07"
-        izz="5.54170402685473E-05" />
+      <inertia ixx="0.00004661" ixy="-0.00000101" ixz="0.00000131"
+             iyy="0.00012523" iyz="0.00000006"
+             izz="0.00010857" />
     </inertial>
     <visual>
@@ -814,5 +758,5 @@
       upper="0"
       effort="1000"
-      velocity="0" />
+      velocity="0.1" />
   </joint>
   <insert_transmission name="l_ank_pitch"/>
@@ -825,11 +769,7 @@
       <mass
         value="0.0443088669743472" />
-      <inertia
-        ixx="3.98750519227104E-05"
-        ixy="8.27728807804659E-11"
-        ixz="3.17919598040036E-09"
-        iyy="5.39463274407849E-05"
-        iyz="-3.77243123537462E-08"
-        izz="1.97495395193279E-05" />
+      <inertia ixx="0.00004034" ixy="-0.00000019" ixz="0.00000012"
+             iyy="0.00007874" iyz="0.00000101"
+             izz="0.00011579" />
     </inertial>
     <visual>
@@ -873,5 +813,5 @@
       upper="0"
       effort="1000"
-      velocity="0" />
+      velocity="0.1" />
   </joint>
   <insert_transmission name="l_ank_roll"/>
@@ -885,11 +825,7 @@
       <mass
         value="0.0229829364852389" />
-      <inertia
-        ixx="1.43427059428118E-05"
-        ixy="8.27728850397696E-11"
-        ixz="1.78618118586269E-10"
-        iyy="1.40196878929159E-05"
-        iyz="3.77243123518229E-08"
-        izz="5.34102862853243E-06" />
+      <inertia ixx="0.00000151" ixy="0.0" ixz="0.00000001"
+             iyy="0.00000430" iyz="0.0"
+             izz="0.00000412" />
     </inertial>
     <visual>
@@ -933,5 +869,5 @@
       upper="0"
       effort="1000"
-      velocity="0" />
+      velocity="0.1" />
   </joint>
   <insert_transmission name="r_hip_yaw"/>
@@ -944,11 +880,7 @@
       <mass
         value="0.151586182496668" />
-      <inertia
-        ixx="5.50281750229322E-05"
-        ixy="8.98440761834266E-07"
-        ixz="1.16956224699704E-12"
-        iyy="3.44253544650064E-05"
-        iyz="-9.07656515072372E-07"
-        izz="5.54170402685471E-05" />
+      <inertia ixx="0.00004661" ixy="0.00000101" ixz="-0.00000131"
+             iyy="0.00012523" iyz="0.00000006"
+             izz="0.00010857" />
     </inertial>
     <visual>
@@ -992,5 +924,5 @@
       upper="0"
       effort="1000"
-      velocity="0" />
+      velocity="0.1" />
   </joint>
   <insert_transmission name="r_hip_roll"/>
@@ -1003,11 +935,7 @@
       <mass
         value="0.100631639038866" />
-      <inertia
-        ixx="4.17310749465033E-05"
-        ixy="-9.08752859615629E-07"
-        ixz="5.42245635045147E-09"
-        iyy="3.21411717550871E-05"
-        iyz="6.05551462761427E-07"
-        izz="5.70627485423264E-05" />
+      <inertia ixx="0.00010499" ixy="0.00000001" ixz="-0.00000071"
+             iyy="0.00009613" iyz="-0.00000353"
+             izz="0.00002493" />
     </inertial>
     <visual>
@@ -1051,5 +979,5 @@
       upper="0"
       effort="1000"
-      velocity="0" />
+      velocity="0.1" />
   </joint>
   <insert_transmission name="r_hip_pitch"/>
@@ -1062,11 +990,7 @@
       <mass
         value="0.0624359207391501" />
-      <inertia
-        ixx="0.000103909612579586"
-        ixy="2.24696234577128E-10"
-        ixz="1.61509844866009E-10"
-        iyy="4.75106496264916E-05"
-        iyz="-1.78798066876231E-05"
-        izz="0.000119654238933633" />
+      <inertia ixx="0.00003715" ixy="0.0" ixz="0.0"
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
Commit message: change joint revolute

File: rscuad_description/urdf/rscuad.xacro (robot description, xacro)
@@ -83,5 +83,5 @@
   <joint
     name="head_pan"
-    type="continuous">
+    type="revolute">
     <origin
       xyz="0.035958 -0.1394 0.14298"
@@ -93,9 +93,5 @@
     <axis
       xyz="0 1 0" />
-    <limit
-      lower="0"
-      upper="0"
-      effort="50"
-      velocity="0.1" />
+     <limit effort="1000" velocity="10" lower="${-pi*0.9}" upper="${pi*0.9}" />
   </joint>
   <insert_transmission name="head_pan"/>
@@ -138,5 +134,5 @@
   <joint
     name="head_tilt"
-    type="continuous">
+    type="revolute">
     <origin
       xyz="0 -0.0285 0.01"
@@ -148,9 +144,5 @@
     <axis
       xyz="-1 0 0" />
-    <limit
-      lower="0"
-      upper="0"
-      effort="50"
-      velocity="0.1" />
+     <limit effort="1000" velocity="10" lower="${-pi*0.9}" upper="${pi*0.9}" />
   </joint>
   <insert_transmission name="head_tilt"/>
@@ -194,5 +186,5 @@
   <joint
     name="l_sho_pitch"
-    type="continuous">
+    type="revolute">
     <origin
       xyz="0.10096 -0.1394 0.12423"
@@ -204,9 +196,5 @@
     <axis
       xyz="-1 0 0" />
-    <limit
-      lower="0"
-      upper="0"
-      effort="100"
-      velocity="0.1" />
+     <limit effort="1000" velocity="10" lower="${-pi*0.9}" upper="${pi*0.9}" />
   </joint>
   <insert_transmission name="l_sho_pitch"/>
@@ -249,5 +237,5 @@
   <joint
     name="l_sho_roll"
-    type="continuous">
+    type="revolute">
     <origin
       xyz="0.0385 -0.01 0"
@@ -259,9 +247,5 @@
     <axis
       xyz="0 0 -1" />
-    <limit
-      lower="0"
-      upper="0"
-      effort="1000"
-      velocity="0.1" />
+    <limit effort="1000" velocity="10" lower="${-pi*0.9}" upper="${pi*0.9}" />
   </joint>
   <insert_transmission name="l_sho_roll"/>
@@ -304,5 +288,5 @@
   <joint
     name="l_el"
-    type="continuous">
+    type="revolute">
     <origin
       xyz="0.0874466726391421 0 0.0100000000000002"
@@ -314,9 +298,5 @@
     <axis
       xyz="0 -1 0" />
-    <limit
-      lower="0"
-      upper="0"
-      effort="1000"
-      velocity="0.1" />
+     <limit effort="1000" velocity="10" lower="${-pi*0.9}" upper="${pi*0.9}" />
   </joint>
   <insert_transmission name="l_el"/>
@@ -360,5 +340,5 @@
   <joint
     name="r_sho_pitch"
-    type="continuous">
+    type="revolute">
     <origin
       xyz="-0.0290205030447131 -0.139400454049433 0.124229542783902"
@@ -370,9 +350,5 @@
     <axis
       xyz="-1 0 0" />
-    <limit
-      lower="0"
-      upper="0"
-      effort="1000"
-      velocity="0.1" />
+     <limit effort="1000" velocity="10" lower="${-pi*0.9}" upper="${pi*0.9}" />
   </joint>
   <insert_transmission name="r_sho_pitch"/>
@@ -415,5 +391,5 @@
   <joint
     name="r_sho_roll"
-    type="continuous">
+    type="revolute">
     <origin
       xyz="-0.0384999999999999 -0.00999999999999629 0"
@@ -425,9 +401,5 @@
     <axis
       xyz="0 0 -1" />
-    <limit
-      lower="0"
-      upper="0"
-      effort="1000"
-      velocity="0.1" />
+     <limit effort="1000" velocity="10" lower="${-pi*0.9}" upper="${pi*0.9}" />
   </joint>
   <insert_transmission name="r_sho_roll"/>
@@ -470,5 +442,5 @@
   <joint
     name="r_el"
-    type="continuous">
+    type="revolute">
     <origin
       xyz="-0.0936500000000009 0 0.0099999999999961"
@@ -480,9 +452,5 @@
     <axis
       xyz="0 -1 0" />
-    <limit
-      lower="0"
-      upper="0"
-      effort="1000"
-      velocity="0.1" />
+     <limit effort="1000" velocity="10" lower="${-pi*0.9}" upper="${pi*0.9}" />
   </joint>
   <insert_transmission name="r_el"/>
@@ -526,5 +494,5 @@
   <joint
     name="l_hip_yaw"
-    type="continuous">
+    type="revolute">
     <origin
       xyz="0.0809483118859766 -0.13794445404943 0.00675246433967373"
@@ -536,9 +504,5 @@
     <axis
       xyz="0 -1 0" />
-    <limit
-      lower="0"
-      upper="0"
-      effort="1000"
-      velocity="0.1" />
+     <limit effort="1000" velocity="10" lower="${-pi*0.9}" upper="${pi*0.9}" />
   </joint>
   <insert_transmission name="l_hip_yaw"/>
@@ -581,5 +545,5 @@
   <joint
     name="l_hip_roll"
-    type="continuous">
+    type="revolute">
     <origin
       xyz="0 -0.0360348499633859 0"
@@ -591,9 +555,5 @@
     <axis
       xyz="0 0 -1" />
-    <limit
-      lower="0"
-      upper="0"
-      effort="1000"
-      velocity="0.1" />
+     <limit effort="1000" velocity="10" lower="${-pi*0.9}" upper="${pi*0.9}" />
   </joint>
   <insert_transmission name="l_hip_roll"/>
@@ -636,8 +596,8 @@
   <joint
     name="l_hip_pitch"
-    type="continuous">
+    type="revolute">
     <origin
       xyz="0 0 -0.000599999999901152"
-      rpy="0 0 0" />
+      rpy="-0.3 0 0" />
     <parent
       link="l_hip_roll" />
@@ -646,9 +606,5 @@
     <axis
       xyz="-1 0 0" />
-    <limit
-      lower="0"
-      upper="0"
-      effort="1000"
-      velocity="0.1" />
+     <limit effort="1000" velocity="10" lower="${-pi*0.9}" upper="${pi*0.9}" />
   </joint>
   <insert_transmission name="l_hip_pitch"/>
@@ -691,8 +647,8 @@
   <joint
     name="l_knee"
-    type="continuous">
+    type="revolute">
     <origin
       xyz="0 -0.121999999999998 -3.60787874466861E-05"
-      rpy="0 0 0" />
+      rpy="0.5 0 0" />
     <parent
       link="l_hip_pitch" />
@@ -701,9 +657,5 @@
     <axis
       xyz="-1 0 0" />
-    <limit
-      lower="0"
-      upper="0"
-      effort="1000"
-      velocity="0.1" />
+     <limit effort="1000" velocity="10" lower="${-pi*0.9}" upper="${pi*0.9}" />
   </joint>
   <insert_transmission name="l_knee"/>
@@ -746,8 +698,8 @@
   <joint
     name="l_ank_pitch"
-    type="continuous">
+    type="revolute">
     <origin
       xyz="0 -0.12200007459305 0.000539974593052855"
-      rpy="0 0 -3.14159265358979" />
+      rpy="0.5 0 -3.14159265358979" />
     <parent
       link="l_knee" />
@@ -756,9 +708,5 @@
     <axis
       xyz="1 0 0" />
-    <limit
-      lower="0"
-      upper="0"
-      effort="1000"
-      velocity="0.1" />
+     <limit effort="1000" velocity="10" lower="${-pi*0.9}" upper="${pi*0.9}" />
   </joint>
   <insert_transmission name="l_ank_pitch"/>
@@ -801,5 +749,5 @@
   <joint
     name="l_ank_roll"
-    type="continuous">
+    type="revolute">
     <origin
       xyz="0 0 0"
@@ -811,9 +759,5 @@
     <axis
       xyz="0 0 -1" />
-    <limit
-      lower="0"
-      upper="0"
-      effort="1000"
-      velocity="0.1" />
+     <limit effort="1000" velocity="10" lower="${-pi*0.9}" upper="${pi*0.9}" />
   </joint>
   <insert_transmission name="l_ank_roll"/>
@@ -857,5 +801,5 @@
   <joint
     name="r_hip_yaw"
-    type="continuous">
+    type="revolute">
     <origin
       xyz="-0.00903979651901684 -0.13794425404943 0.00679279956234802"
@@ -867,9 +811,5 @@
     <axis
       xyz="0 -1 0" />
-    <limit
-      lower="0"
-      upper="0"
-      effort="1000"
-      velocity="0.1" />
+     <limit effort="1000" velocity="10" lower="${-pi*0.9}" upper="${pi*0.9}" />
   </joint>
   <insert_transmission name="r_hip_yaw"/>
@@ -912,5 +852,5 @@
   <joint
     name="r_hip_roll"
-    type="continuous">
+    type="revolute">
     <origin
       xyz="0 -0.0360348499633864 0"
@@ -922,9 +862,5 @@
     <axis
       xyz="0 0 -1" />
-    <limit
-      lower="0"
-      upper="0"
-      effort="1000"
-      velocity="0.1" />
+     <limit effort="1000" velocity="10" lower="${-pi*0.9}" upper="${pi*0.9}" />
   </joint>
   <insert_transmission name="r_hip_roll"/>
@@ -967,8 +903,8 @@
   <joint
     name="r_hip_pitch"
-    type="continuous">
+    type="revolute">
     <origin
       xyz="0 0 -0.000599999999901429"
-      rpy="0 0 0" />
+      rpy="-0.3 0 0" />
     <parent
       link="r_hip_roll" />
@@ -977,9 +913,5 @@
     <axis
       xyz="-1 0 0" />
-    <limit
-      lower="0"
-      upper="0"
-      effort="1000"
-      velocity="0.1" />
+     <limit effort="1000" velocity="10" lower="${-pi*0.9}" upper="${pi*0.9}" />
   </joint>
   <insert_transmission name="r_hip_pitch"/>
@@ -1022,8 +954,8 @@
   <joint
     name="r_knee"
-    type="continuous">
+    type="revolute">
     <origin
       xyz="0 -0.121999999999998 -3.60787874468527E-05"
-      rpy="0 0 0" />
+      rpy="0.5 0 0" />
     <parent
       link="r_hip_pitch" />
@@ -1032,9 +964,5 @@
     <axis
       xyz="-1 0 0" />
-    <limit
-      lower="0"
-      upper="0"
-      effort="1000"
-      velocity="0.1" />
+     <limit effort="1000" velocity="10" lower="${-pi*0.9}" upper="${pi*0.9}" />
   </joint>
   <insert_transmission name="r_knee"/>
@@ -1077,8 +1005,8 @@
   <joint
     name="r_ank_pitch"
-    type="continuous">
+    type="revolute">
     <origin
       xyz="0 -0.122 0.00053997"
-      rpy="0 0 -3.1416" />
+      rpy="0.5 0 -3.1416" />
     <parent
       link="r_knee" />
@@ -1087,9 +1015,5 @@
     <axis
       xyz="1 0 0" />
-    <limit
-      lower="0"
-      upper="0"
-      effort="1000"
-      velocity="0.1" />
+     <limit effort="1000" velocity="10" lower="${-pi*0.9}" upper="${pi*0.9}" />
   </joint>
   <insert_transmission name="r_ank_pitch"/>
@@ -1132,5 +1056,5 @@
   <joint
     name="r_ank_roll"
-    type="continuous">
+    type="revolute">
     <origin
       xyz="0 0 0"
@@ -1142,9 +1066,5 @@
     <axis
       xyz="0 0 -1" />
-    <limit
-      lower="0"
-      upper="0"
-      effort="1000"
-      velocity="0.1" />
+     <limit effort="1000" velocity="10" lower="${-pi*0.9}" upper="${pi*0.9}" />
   </joint>
   <insert_transmission name="r_ank_roll"/>

Commit message: fix running IK, but not normal

File: rscuad_description/urdf/rscuad.xacro (robot description, xacro)
@@ -963,5 +963,6 @@
       link="r_knee" />
     <axis
-      xyz="-1 0 0" />
+      xyz="1 0 0" />
+    <!-- <limit effort="1000" velocity="100" lower="${-pi*0.9}" upper="${pi*0.9}" /> -->
      <limit effort="1000" velocity="10" lower="${-pi*0.9}" upper="${pi*0.9}" />
   </joint>
