Commit message: value reduction inertia & fix ankle position

File: rscuad_description/urdf/rscuad.xacro (robot description, xacro)
@@ -93,5 +93,5 @@
     <axis
       xyz="0 1 0" />
-     <limit effort="1000" velocity="10" lower="${-pi*0.9}" upper="${pi*0.9}" />
+     <limit effort="100" velocity="1" lower="${-pi*0.9}" upper="${pi*0.9}" />
   </joint>
   <insert_transmission name="head_pan"/>
@@ -144,5 +144,5 @@
     <axis
       xyz="-1 0 0" />
-     <limit effort="1000" velocity="10" lower="${-pi*0.9}" upper="${pi*0.9}" />
+     <limit effort="100" velocity="1" lower="${-pi*0.9}" upper="${pi*0.9}" />
   </joint>
   <insert_transmission name="head_tilt"/>
@@ -196,5 +196,5 @@
     <axis
       xyz="-1 0 0" />
-     <limit effort="1000" velocity="10" lower="${-pi*0.9}" upper="${pi*0.9}" />
+     <limit effort="100" velocity="1" lower="${-pi*0.9}" upper="${pi*0.9}" />
   </joint>
   <insert_transmission name="l_sho_pitch"/>
@@ -247,5 +247,5 @@
     <axis
       xyz="0 0 -1" />
-    <limit effort="1000" velocity="10" lower="${-pi*0.9}" upper="${pi*0.9}" />
+    <limit effort="100" velocity="1" lower="${-pi*0.9}" upper="${pi*0.9}" />
   </joint>
   <insert_transmission name="l_sho_roll"/>
@@ -298,5 +298,5 @@
     <axis
       xyz="0 -1 0" />
-     <limit effort="1000" velocity="10" lower="${-pi*0.9}" upper="${pi*0.9}" />
+     <limit effort="100" velocity="1" lower="${-pi*0.9}" upper="${pi*0.9}" />
   </joint>
   <insert_transmission name="l_el"/>
@@ -350,5 +350,5 @@
     <axis
       xyz="-1 0 0" />
-     <limit effort="1000" velocity="10" lower="${-pi*0.9}" upper="${pi*0.9}" />
+     <limit effort="100" velocity="1" lower="${-pi*0.9}" upper="${pi*0.9}" />
   </joint>
   <insert_transmission name="r_sho_pitch"/>
@@ -401,5 +401,5 @@
     <axis
       xyz="0 0 -1" />
-     <limit effort="1000" velocity="10" lower="${-pi*0.9}" upper="${pi*0.9}" />
+     <limit effort="100" velocity="1" lower="${-pi*0.9}" upper="${pi*0.9}" />
   </joint>
   <insert_transmission name="r_sho_roll"/>
@@ -452,5 +452,5 @@
     <axis
       xyz="0 -1 0" />
-     <limit effort="1000" velocity="10" lower="${-pi*0.9}" upper="${pi*0.9}" />
+     <limit effort="100" velocity="1" lower="${-pi*0.9}" upper="${pi*0.9}" />
   </joint>
   <insert_transmission name="r_el"/>
@@ -504,5 +504,5 @@
     <axis
       xyz="0 -1 0" />
-     <limit effort="1000" velocity="10" lower="${-pi*0.9}" upper="${pi*0.9}" />
+     <limit effort="100" velocity="1" lower="${-pi*0.9}" upper="${pi*0.9}" />
   </joint>
   <insert_transmission name="l_hip_yaw"/>
@@ -555,5 +555,5 @@
     <axis
       xyz="0 0 -1" />
-     <limit effort="1000" velocity="10" lower="${-pi*0.9}" upper="${pi*0.9}" />
+     <limit effort="100" velocity="1" lower="${-pi*0.9}" upper="${pi*0.9}" />
   </joint>
   <insert_transmission name="l_hip_roll"/>
@@ -606,5 +606,5 @@
     <axis
       xyz="-1 0 0" />
-     <limit effort="1000" velocity="10" lower="${-pi*0.9}" upper="${pi*0.9}" />
+     <limit effort="100" velocity="1" lower="${-pi*0.9}" upper="${pi*0.9}" />
   </joint>
   <insert_transmission name="l_hip_pitch"/>
@@ -657,5 +657,5 @@
     <axis
       xyz="-1 0 0" />
-     <limit effort="1000" velocity="10" lower="${-pi*0.9}" upper="${pi*0.9}" />
+     <limit effort="100" velocity="1" lower="${-pi*0.9}" upper="${pi*0.9}" />
   </joint>
   <insert_transmission name="l_knee"/>
@@ -708,5 +708,5 @@
     <axis
       xyz="1 0 0" />
-     <limit effort="1000" velocity="10" lower="${-pi*0.9}" upper="${pi*0.9}" />
+     <limit effort="100" velocity="1" lower="${-pi*0.9}" upper="${pi*0.9}" />
   </joint>
   <insert_transmission name="l_ank_pitch"/>
@@ -759,5 +759,5 @@
     <axis
       xyz="0 0 -1" />
-     <limit effort="1000" velocity="10" lower="${-pi*0.9}" upper="${pi*0.9}" />
+     <limit effort="100" velocity="1" lower="${-pi*0.9}" upper="${pi*0.9}" />
   </joint>
   <insert_transmission name="l_ank_roll"/>
@@ -811,5 +811,5 @@
     <axis
       xyz="0 -1 0" />
-     <limit effort="1000" velocity="10" lower="${-pi*0.9}" upper="${pi*0.9}" />
+     <limit effort="100" velocity="1" lower="${-pi*0.9}" upper="${pi*0.9}" />
   </joint>
   <insert_transmission name="r_hip_yaw"/>
@@ -862,5 +862,5 @@
     <axis
       xyz="0 0 -1" />
-     <limit effort="1000" velocity="10" lower="${-pi*0.9}" upper="${pi*0.9}" />
+     <limit effort="100" velocity="1" lower="${-pi*0.9}" upper="${pi*0.9}" />
   </joint>
   <insert_transmission name="r_hip_roll"/>
@@ -913,5 +913,5 @@
     <axis
       xyz="-1 0 0" />
-     <limit effort="1000" velocity="10" lower="${-pi*0.9}" upper="${pi*0.9}" />
+     <limit effort="100" velocity="1" lower="${-pi*0.9}" upper="${pi*0.9}" />
   </joint>
   <insert_transmission name="r_hip_pitch"/>
@@ -964,6 +964,6 @@
     <axis
       xyz="1 0 0" />
-    <!-- <limit effort="1000" velocity="100" lower="${-pi*0.9}" upper="${pi*0.9}" /> -->
-     <limit effort="1000" velocity="10" lower="${-pi*0.9}" upper="${pi*0.9}" />
+    <!-- <limit effort="100" velocity="10" lower="${-pi*0.9}" upper="${pi*0.9}" /> -->
+     <limit effort="100" velocity="1" lower="${-pi*0.9}" upper="${pi*0.9}" />
   </joint>
   <insert_transmission name="r_knee"/>
@@ -1016,5 +1016,5 @@
     <axis
       xyz="1 0 0" />
-     <limit effort="1000" velocity="10" lower="${-pi*0.9}" upper="${pi*0.9}" />
+     <limit effort="100" velocity="1" lower="${-pi*0.9}" upper="${pi*0.9}" />
   </joint>
   <insert_transmission name="r_ank_pitch"/>
@@ -1067,5 +1067,5 @@
     <axis
       xyz="0 0 -1" />
-     <limit effort="1000" velocity="10" lower="${-pi*0.9}" upper="${pi*0.9}" />
+     <limit effort="100" velocity="1" lower="${-pi*0.9}" upper="${pi*0.9}" />
   </joint>
   <insert_transmission name="r_ank_roll"/>

Commit message: done position robot

File: rscuad_description/urdf/rscuad.xacro (robot description, xacro)
@@ -6,4 +6,6 @@
 update 3 june
 value reduction op3
+update 6 june
+value reduction mess rscuad
 -->
 <robot name="rscuad" xmlns:xacro="http://www.ros.org/wiki/xacro">
@@ -18,5 +20,5 @@
         rpy="0 0 0" />
       <mass
-        value="0.845681147773924" />
+        value="0.0045681147773924" />
       <inertia ixx="0.00340499" ixy="0.00000572" ixz="-0.00004256"
              iyy="0.00296939" iyz="-0.00000059"
@@ -54,5 +56,5 @@
         rpy="0 0 0" />
       <mass
-        value="0.0127468700670499" />
+        value="0.00127468700670499" />
       <inertia ixx="0.00000397" ixy="0.0" ixz="-0.00000031"
              iyy="0.00000165" iyz="0.0"
@@ -95,5 +97,5 @@
     <axis
       xyz="0 1 0" />
-     <limit effort="100" velocity="1" lower="${-pi*0.9}" upper="${pi*0.9}" />
+     <limit effort="1000" velocity="1" lower="${-pi*0.9}" upper="${pi*0.9}" />
   </joint>
   <insert_transmission name="head_pan"/>
@@ -105,5 +107,5 @@
         rpy="0 0 0" />
       <mass
-        value="0.12573924511903" />
+        value="0.0012573924511903" />
       <inertia ixx="0.00010612" ixy="0.00000011" ixz="-0.00000910"
              iyy="0.00008721" iyz="0.00000084"
@@ -146,5 +148,5 @@
     <axis
       xyz="-1 0 0" />
-     <limit effort="100" velocity="1" lower="${-pi*0.9}" upper="${pi*0.9}" />
+     <limit effort="1000" velocity="1" lower="${-pi*0.9}" upper="${pi*0.9}" />
   </joint>
   <insert_transmission name="head_tilt"/>
@@ -198,5 +200,5 @@
     <axis
       xyz="-1 0 0" />
-     <limit effort="100" velocity="1" lower="${-pi*0.9}" upper="${pi*0.9}" />
+     <limit effort="1000" velocity="1" lower="${-pi*0.9}" upper="${pi*0.9}" />
   </joint>
   <insert_transmission name="l_sho_pitch"/>
@@ -208,5 +210,5 @@
         rpy="0 0 0" />
       <mass
-        value="0.0884003305596694" />
+        value="0.0284003305596694" />
       <inertia ixx="0.00022804" ixy="-0.00000001" ixz="0.00000003"
              iyy="0.00003042" iyz="0.00000059"
@@ -249,5 +251,5 @@
     <axis
       xyz="0 0 -1" />
-    <limit effort="100" velocity="1" lower="${-pi*0.9}" upper="${pi*0.9}" />
+    <limit effort="1000" velocity="1" lower="${-pi*0.9}" upper="${pi*0.9}" />
   </joint>
   <insert_transmission name="l_sho_roll"/>
@@ -300,5 +302,5 @@
     <axis
       xyz="0 -1 0" />
-     <limit effort="100" velocity="1" lower="${-pi*0.9}" upper="${pi*0.9}" />
+     <limit effort="1000" velocity="1" lower="${-pi*0.9}" upper="${pi*0.9}" />
   </joint>
   <insert_transmission name="l_el"/>
@@ -352,5 +354,5 @@
     <axis
       xyz="-1 0 0" />
-     <limit effort="100" velocity="1" lower="${-pi*0.9}" upper="${pi*0.9}" />
+     <limit effort="1000" velocity="1" lower="${-pi*0.9}" upper="${pi*0.9}" />
   </joint>
   <insert_transmission name="r_sho_pitch"/>
@@ -362,5 +364,5 @@
         rpy="0 0 0" />
       <mass
-        value="0.0884003307974895" />
+        value="0.0284003307974895" />
       <inertia ixx="0.00022804" ixy="0.00000001" ixz="0.00000003"
              iyy="0.00003042" iyz="-0.00000059"
@@ -403,5 +405,5 @@
     <axis
       xyz="0 0 -1" />
-     <limit effort="100" velocity="1" lower="${-pi*0.9}" upper="${pi*0.9}" />
+     <limit effort="1000" velocity="1" lower="${-pi*0.9}" upper="${pi*0.9}" />
   </joint>
   <insert_transmission name="r_sho_roll"/>
@@ -454,5 +456,5 @@
     <axis
       xyz="0 -1 0" />
-     <limit effort="100" velocity="1" lower="${-pi*0.9}" upper="${pi*0.9}" />
+     <limit effort="1000" velocity="1" lower="${-pi*0.9}" upper="${pi*0.9}" />
   </joint>
   <insert_transmission name="r_el"/>
@@ -506,5 +508,5 @@
     <axis
       xyz="0 -1 0" />
-     <limit effort="100" velocity="1" lower="${-pi*0.9}" upper="${pi*0.9}" />
+     <limit effort="1000" velocity="1" lower="${-pi*0.9}" upper="${pi*0.9}" />
   </joint>
   <insert_transmission name="l_hip_yaw"/>
@@ -516,5 +518,5 @@
         rpy="0 0 0" />
       <mass
-        value="0.151586182496668" />
+        value="0.0151586182496668" />
       <inertia ixx="0.00004661" ixy="-0.00000101" ixz="-0.00000131"
              iyy="0.00012523" iyz="-0.00000006"
@@ -557,5 +559,5 @@
     <axis
       xyz="0 0 -1" />
-     <limit effort="100" velocity="1" lower="${-pi*0.9}" upper="${pi*0.9}" />
+     <limit effort="1000" velocity="1" lower="${-pi*0.9}" upper="${pi*0.9}" />
   </joint>
   <insert_transmission name="l_hip_roll"/>
@@ -567,5 +569,5 @@
         rpy="0 0 0" />
       <mass
-        value="0.100631639038866" />
+        value="0.0100631639038866" />
       <inertia ixx="0.00010499" ixy="-0.00000001" ixz="-0.00000071"
              iyy="0.00009613" iyz="0.00000353"
@@ -608,5 +610,5 @@
     <axis
       xyz="-1 0 0" />
-     <limit effort="100" velocity="1" lower="${-pi*0.9}" upper="${pi*0.9}" />
+     <limit effort="1000" velocity="1" lower="${-pi*0.9}" upper="${pi*0.9}" />
   </joint>
   <insert_transmission name="l_hip_pitch"/>
@@ -659,5 +661,5 @@
     <axis
       xyz="-1 0 0" />
-     <limit effort="100" velocity="1" lower="${-pi*0.9}" upper="${pi*0.9}" />
+     <limit effort="1000" velocity="1" lower="${-pi*0.9}" upper="${pi*0.9}" />
   </joint>
   <insert_transmission name="l_knee"/>
@@ -669,5 +671,5 @@
         rpy="0 0 0" />
       <mass
-        value="0.151586182496668" />
+        value="0.0151586182496668" />
       <inertia ixx="0.00004661" ixy="-0.00000101" ixz="0.00000131"
              iyy="0.00012523" iyz="0.00000006"
@@ -710,5 +712,5 @@
     <axis
       xyz="1 0 0" />
-     <limit effort="100" velocity="1" lower="${-pi*0.9}" upper="${pi*0.9}" />
+     <limit effort="1000" velocity="1" lower="${-pi*0.9}" upper="${pi*0.9}" />
   </joint>
   <insert_transmission name="l_ank_pitch"/>
@@ -761,5 +763,5 @@
     <axis
       xyz="0 0 -1" />
-     <limit effort="100" velocity="1" lower="${-pi*0.9}" upper="${pi*0.9}" />
+     <limit effort="1000" velocity="1" lower="${-pi*0.9}" upper="${pi*0.9}" />
   </joint>
   <insert_transmission name="l_ank_roll"/>
@@ -813,5 +815,5 @@
     <axis
       xyz="0 -1 0" />
-     <limit effort="100" velocity="1" lower="${-pi*0.9}" upper="${pi*0.9}" />
+     <limit effort="1000" velocity="1" lower="${-pi*0.9}" upper="${pi*0.9}" />
   </joint>
   <insert_transmission name="r_hip_yaw"/>
@@ -823,5 +825,5 @@
         rpy="0 0 0" />
       <mass
-        value="0.151586182496668" />
+        value="0.0151586182496668" />
       <inertia ixx="0.00004661" ixy="0.00000101" ixz="-0.00000131"
              iyy="0.00012523" iyz="0.00000006"
@@ -864,5 +866,5 @@
     <axis
       xyz="0 0 -1" />
-     <limit effort="100" velocity="1" lower="${-pi*0.9}" upper="${pi*0.9}" />
+     <limit effort="1000" velocity="1" lower="${-pi*0.9}" upper="${pi*0.9}" />
   </joint>
   <insert_transmission name="r_hip_roll"/>
@@ -874,5 +876,5 @@
         rpy="0 0 0" />
       <mass
-        value="0.100631639038866" />
+        value="0.0100631639038866" />
       <inertia ixx="0.00010499" ixy="0.00000001" ixz="-0.00000071"
              iyy="0.00009613" iyz="-0.00000353"
@@ -915,5 +917,5 @@
     <axis
       xyz="-1 0 0" />
-     <limit effort="100" velocity="1" lower="${-pi*0.9}" upper="${pi*0.9}" />
+     <limit effort="1000" velocity="1" lower="${-pi*0.9}" upper="${pi*0.9}" />
   </joint>
   <insert_transmission name="r_hip_pitch"/>
@@ -966,6 +968,6 @@
     <axis
       xyz="1 0 0" />
-    <!-- <limit effort="100" velocity="10" lower="${-pi*0.9}" upper="${pi*0.9}" /> -->
-     <limit effort="100" velocity="1" lower="${-pi*0.9}" upper="${pi*0.9}" />
+    <!-- <limit effort="1000" velocity="10" lower="${-pi*0.9}" upper="${pi*0.9}" /> -->
+     <limit effort="1000" velocity="1" lower="${-pi*0.9}" upper="${pi*0.9}" />
   </joint>
   <insert_transmission name="r_knee"/>
@@ -977,5 +979,5 @@
         rpy="0 0 0" />
       <mass
-        value="0.151586182496669" />
+        value="0.0151586182496669" />
       <inertia ixx="0.00004661" ixy="0.00000101" ixz="0.00000131"
              iyy="0.00012523" iyz="-0.00000006"
@@ -1018,5 +1020,5 @@
     <axis
       xyz="1 0 0" />
-     <limit effort="100" velocity="1" lower="${-pi*0.9}" upper="${pi*0.9}" />
+     <limit effort="1000" velocity="1" lower="${-pi*0.9}" upper="${pi*0.9}" />
   </joint>
   <insert_transmission name="r_ank_pitch"/>
@@ -1069,5 +1071,5 @@
     <axis
       xyz="0 0 -1" />
-     <limit effort="100" velocity="1" lower="${-pi*0.9}" upper="${pi*0.9}" />
+     <limit effort="1000" velocity="1" lower="${-pi*0.9}" upper="${pi*0.9}" />
   </joint>
   <insert_transmission name="r_ank_roll"/>

Commit message: add harness

File: rscuad_description/urdf/rscuad.xacro (robot description, xacro)
@@ -13,4 +13,20 @@
   <xacro:include filename="$(find rscuad_description)/urdf/rscuad.gazebo" />
   <xacro:include filename="$(find rscuad_description)/urdf/transmission.xacro" />
+  <xacro:include filename="$(find rscuad_description)/urdf/gazebo_harness.xacro" />
+  <xacro:add_sim_harness harnessed_link="body"/>
+  <!-- <link name="world">
+  </link> -->
+  <!-- <joint name="world_fixed" type="fixed">
+    <origin xyz="0 0 0" rpy="0 0 0"/>
+    <parent link="world"/>
+    <child link="base"/>
+  </joint> -->
+  <!-- <link name="base">
+  </link>
+  <joint name="base_fixed" type="fixed">
+    <origin xyz="0 0 0" rpy="0 0 0"/>
+    <parent link="base"/>
+    <child link="body"/>
+  </joint> -->
   <link
     name="body">

Commit message: set init and walking | pid setting and fix COG body

File: rscuad_description/urdf/rscuad.xacro (robot description, xacro)
@@ -33,10 +33,10 @@
     <inertial>
       <origin
-        xyz="0.0357056190627579 0.0719364874349917 0.124774491029847"
-        rpy="0 0 0" />
-      <mass
-        value="0.0125681147773924" />
+        xyz="0.0357056190627579 -0.129364874349917 0.124774491029847"
+        rpy="0 0 0" />
+      <mass
+        value="0.0845681147773924" />
       <inertia ixx="0.00340499" ixy="0.00000572" ixz="-0.00004256"
-             iyy="0.00296939" iyz="-0.00000059"
+             iyy="0.296939" iyz="-0.00000059"
              izz="0.00317331" />
     </inertial>
@@ -123,5 +123,5 @@
         rpy="0 0 0" />
       <mass
-        value="0.0012573924511903" />
+        value="0.012573924511903" />
       <inertia ixx="0.00010612" ixy="0.00000011" ixz="-0.00000910"
              iyy="0.00008721" iyz="0.00000084"
@@ -226,5 +226,5 @@
         rpy="0 0 0" />
       <mass
-        value="0.0284003305596694" />
+        value="0.0884003305596694" />
       <inertia ixx="0.00022804" ixy="-0.00000001" ixz="0.00000003"
              iyy="0.00003042" iyz="0.00000059"
@@ -380,5 +380,5 @@
         rpy="0 0 0" />
       <mass
-        value="0.0284003307974895" />
+        value="0.0884003307974895" />
       <inertia ixx="0.00022804" ixy="0.00000001" ixz="0.00000003"
              iyy="0.00003042" iyz="-0.00000059"
