Commit message: fix walking

File: RSCUAD-Common/rscuad_description/urdf/rscuad.xacro (robot description, xacro)
@@ -14,13 +14,13 @@
   <xacro:include filename="$(find rscuad_description)/urdf/transmission.xacro" />
   <xacro:include filename="$(find rscuad_description)/urdf/gazebo_harness.xacro" />
-  <!-- <xacro:add_sim_harness harnessed_link="body"/> -->
-  <!-- <link name="world">
-  </link> -->
-  <!-- <joint name="world_fixed" type="fixed">
+  <xacro:add_sim_harness harnessed_link="body"/>
+  <link name="world">
+  </link>
+  <joint name="world_fixed" type="fixed">
     <origin xyz="0 0 0" rpy="0 0 0"/>
     <parent link="world"/>
     <child link="base"/>
-  </joint> -->
-  <!-- <link name="base">
+  </joint>
+  <link name="base">
   </link>
   <joint name="base_fixed" type="fixed">
@@ -28,5 +28,5 @@
     <parent link="base"/>
     <child link="body"/>
-  </joint> -->
+  </joint>
   <link
     name="body">

Commit message: approach initial robot & gazebo

File: RSCUAD-Common/rscuad_description/urdf/rscuad.xacro (robot description, xacro)
@@ -15,5 +15,5 @@
   <xacro:include filename="$(find rscuad_description)/urdf/gazebo_harness.xacro" />
   <xacro:add_sim_harness harnessed_link="body"/>
-  <link name="world">
+  <!-- <link name="world">
   </link>
   <joint name="world_fixed" type="fixed">
@@ -28,5 +28,5 @@
     <parent link="base"/>
     <child link="body"/>
-  </joint>
+  </joint> -->
   <link
     name="body">

Commit message: add camera

File: RSCUAD-Common/rscuad_description/urdf/rscuad.xacro (robot description, xacro)
@@ -8,4 +8,6 @@
 update 6 june
 value reduction mess rscuad
+update 29 july
+add camera
 -->
 <robot name="rscuad" xmlns:xacro="http://www.ros.org/wiki/xacro">
@@ -15,4 +17,6 @@
   <xacro:include filename="$(find rscuad_description)/urdf/gazebo_harness.xacro" />
   <xacro:add_sim_harness harnessed_link="body"/>
+  <xacro:property name="camera_link" value="0.01" /> <!-- Size of square 'camera' box -->
+  <!-- ============== harness initial ================ -->
   <!-- <link name="world">
   </link>
@@ -1090,3 +1094,30 @@
   </joint>
   <insert_transmission name="r_ank_roll"/>
+  <joint name="camera_joint" type="fixed">
+    <axis xyz="0 1 0" />
+    <origin xyz="0.0 0.0500 0.03"
+      rpy="-1.5708 -1.500 0" />
+    <parent link="head_tilt"/>
+    <child link="camera_link"/>
+  </joint>
+  <!-- Camera -->
+  <link name="camera_link">
+    <collision>
+      <origin xyz="0 0 0" rpy="0 0 0"/>
+      <geometry>
+    <box size="${camera_link} ${camera_link} ${camera_link}"/>
+      </geometry>
+    </collision>
+    <visual>
+      <origin xyz="0 0 0" rpy="0 0 0"/>
+      <geometry>
+    <box size="${camera_link} ${camera_link} ${camera_link}"/>
+      </geometry>
+    </visual>
+    <inertial>
+      <mass value="1e-5" />
+      <origin xyz="0 0 0" rpy="0 0 0"/>
+      <inertia ixx="1e-6" ixy="0" ixz="0" iyy="1e-6" iyz="0" izz="1e-6" />
+    </inertial>
+  </link>
 </robot>

Commit message: fix urdf

File: RSCUAD-Common/rscuad_description/urdf/rscuad.xacro (robot description, xacro)
@@ -41,7 +41,7 @@
       <mass
         value="0.0845681147773924" />
-      <inertia ixx="0.00340499" ixy="0.00000572" ixz="-0.00004256"
-             iyy="0.296939" iyz="-0.00000059"
-             izz="0.00317331" />
+      <inertia ixx="0.00340499" ixy="0.00572" ixz="-0.4256"
+             iyy="0.296939" iyz="-0.59"
+             izz="0.0317331" />
     </inertial>
     <visual>
